Commit message: livox_mid360 can be used but xacro need to be modified

File: urdf/livox_mid360.xacro (robot description, xacro)
@@ -58,4 +58,5 @@
     </gazebo>
   </xacro:macro>
+  <![CDATA[ ]]>
   <xacro:macro name="Livox_Mid40" params="visualize:=True name:=livox">
     <link name="${name}_base">
@@ -64,5 +65,5 @@
         <origin xyz="0.00 0 0.0" rpy="0 0 0"/>
         <geometry>
-          <mesh filename="package://livox_laser_simulation/meshes/livox_mid40.dae">
+          <mesh filename="package://livox_laser_simulation/meshes/livox_mid360.dae">
           </mesh>
         </geometry>
@@ -70,8 +71,9 @@
       <collision>
 		  <origin xyz="0 0 0" rpy="0 0 0" /> <geometry> <mesh
-		  filename="package://livox_laser_simulation/meshes/livox_mid40.dae">
+		  filename="package://livox_laser_simulation/meshes/livox_mid360.dae">
 		  </mesh> </geometry>
       </collision>
     </link>
+    <![CDATA[]]>
     <link name="${name}">
       <xacro:null_inertial/>
